File: Hardware/PCB.brd (EAGLE design)
At the start: 170.2 x 111.2 mm, 103 parts, among them IC1 BD5229G-TR, IC4 XC6220A331MR-G, J1 FH34SRJ-24S-0.5SH_99_, J2 SAMACSYS_PARTS_USB4110-GF-A, J3 QWIIC_RIGHT_ANGLE, J4 112A-TAAR-R03_ATTEND, Q1 20V/4.2A/52mΩ/1.4W, Q2 20V/4.2A/52mΩ/1.4W, Q3 SI1308EDL-T1-GE3, U1 W25Q512JVEIQ, U2 ESP32-C6-WROOM-1-N8, U3 DS3231SN#, U4 MAX17048G+T10

Commit message: Solved Issues
Parts:
- C1_BAT1: value (none) -> 4.7uF
- C3: value (none) -> 100uF
- renumbered TP1 to TX, TP10 to SCK, TP11 to EPD_BUSY, TP12 to EPD_CS, TP13 to EPD_DC, TP14 to EPD_RST, TP15 to EPD_3V3_C, TP16 to VBUS, TP17 to INT_RTC, TP2 to RX, TP3 to VBAT, TP4 to GND, TP5 to GND', TP6 to 3V3, TP7 to EPD_3V3, TP8 to MISO, TP9 to MOSI
Routing:
- net SDA: track 202.8 -> 209.6 mm
